File: design/BLDC_4.kicad_pcb (KiCad board)
At the start: 4 copper layers, 38.5 x 65 mm, 127 parts, among them K1 SERVO, P1 HALL/Encoder, P101 CANBUS, P2 SWD, P3 PWR_COMM, P4 IN+, P5 IN-, P6 MOTOR1, P7 MOTOR2, P9 MOTOR3, Q1 IRFS7530, Q2 IRFS7530, Q3 IRFS7530, Q4 IRFS7530, Q5 IRFS7530, Q6 IRFS7530, U1 STM32F40X_LQFP64, U2 TC2117, U3 DRV8302, U401 SN65HVD232, X1 MINI-USB-SHIELD-32005-201, X2 8MHz 10ppm

Commit message: Premier commit après synchronisation du projet
premier commit après avoir synchroniser le projet dans mon espace de travail. plusieurs composants sont inéxistant dans  la librairie. il vas falloir les rajouter par la suite et commit le projet mis a jour
Parts:
- removed 1PIN (x2): P***, 1pin
- removed 1PIN (x2): P***, Connect:1pin
- removed G***: oshw_silkscreen-back_3mm, oshw_silkscreen-back_3mm
Connections:
- net /Filters/TEMP_IN renamed /Filters/TEMP_MOTOR
- net /MCU/MISO_ADC_EXT2 renamed /MISO_RX_SCL
- net /MCU/RX_SCL_MOSI renamed /RX_SCL_MOSI
- net /MCU/SCK_ADC_EXT renamed /SCK_ADC_EXT
- net /MCU/TX_SDA_NSS renamed /TX_SDA
- P2 pad 6: Net-(P2-Pad6) -> unconnected-(P2-Pad6)
- U1 pad 11: Net-(U1-Pad11) -> unconnected-(U1-PC3(ADC123_IN13)-Pad11)
- U1 pad 2: Net-(U1-Pad2) -> unconnected-(U1-PC13_(RTC_AF1)-Pad2)
- U1 pad 28: Net-(U1-Pad28) -> unconnected-(U1-PB2-BOOT1-Pad28)
- U1 pad 3: Net-(U1-Pad3) -> unconnected-(U1-PC14-OSC32_IN-Pad3)
- U1 pad 39: Net-(U1-Pad39) -> unconnected-(U1-PC8-Pad39)
- U1 pad 4: Net-(U1-Pad4) -> unconnected-(U1-PC15-OSC32_OUT-Pad4)
- U1 pad 40: Net-(U1-Pad40) -> unconnected-(U1-PC9-Pad40)
- U1 pad 50: Net-(U1-Pad50) -> unconnected-(U1-PA15(JTDI)-Pad50)
- U1 pad 54: Net-(U1-Pad54) -> unconnected-(U1-PD2-Pad54)
- U1 pad 55: Net-(U1-Pad55) -> unconnected-(U1-PB3(JTDO/TRACESWO)-Pad55)
- U1 pad 56: Net-(U1-Pad56) -> unconnected-(U1-PB4(NJTRST)-Pad56)
- U1 pad 9: Net-(U1-Pad9) -> unconnected-(U1-PC1(ADC123_IN11)-Pad9)
- U3 pad 4: Net-(U3-Pad4) -> unconnected-(U3-PWRGD-Pad4)
- U3 pad 5: Net-(U3-Pad5) -> unconnected-(U3-OCTW-Pad5)
- U3 pad 55: Net-(U3-Pad55) -> unconnected-(U3-EN_BUCK-Pad55)
- U3 pad 56: Net-(U3-Pad56) -> unconnected-(U3-SS_TR-Pad56)
- U401 pad 5: Net-(U401-Pad5) -> unconnected-(U401-Vref-Pad5)
- X1 pad 4: Net-(X1-Pad4) -> unconnected-(X1-Pad4)
Routing:
- added copper zone on In1.Cu, net /Mosfet driver/H1_VS
- added copper zone on In2.Cu, net /Mosfet driver/H1_VS
- added copper zone on In1.Cu, net /Mosfet driver/H2_VS
- added copper zone on In2.Cu, net /Mosfet driver/H2_VS
- added copper zone on In1.Cu, net /Mosfet driver/H3_VS
- added copper zone on In2.Cu, net /Mosfet driver/H3_VS
- added copper zone on In1.Cu, net GND
- added copper zone on In2.Cu, net GND
- removed copper zone on GND, net /Mosfet driver/H1_VS
- removed copper zone on GND2, net /Mosfet driver/H1_VS
- removed copper zone on GND, net /Mosfet driver/H2_VS
- removed copper zone on GND2, net /Mosfet driver/H2_VS
- removed copper zone on GND, net /Mosfet driver/H3_VS
- removed copper zone on GND2, net /Mosfet driver/H3_VS
- removed copper zone on GND, net GND
- removed copper zone on GND2, net GND
Other:
- net class Default removed
